File: XTA-35/XTA-35.kicad_pcb (KiCad board)
At the start: 2 copper layers, 222.1 x 98.7 mm, 27 parts, among them U4 RPI_PICO

Commit message: A bit more board/footprint work.
Parts:
- J1: renamed from REF**; value PinHeader_2x20_P2.54mm_Horizontal -> XTA_Connector
- XTA Power: renamed from conn_hdd_15-24-4441; value JP*** -> J3
Connections:
- net /INIT_DRIVE renamed /BOOT_INTERNAL
- J1 pad 1: (no net) -> ~RESET
- J1 pad 10: (no net) -> GND
- J1 pad 11: (no net) -> D3
- J1 pad 12: (no net) -> GND
- J1 pad 13: (no net) -> D2
- J1 pad 14: (no net) -> GND
- J1 pad 15: (no net) -> D1
- J1 pad 16: (no net) -> GND
- J1 pad 17: (no net) -> D0
- J1 pad 18: (no net) -> GND
- J1 pad 19: (no net) -> GND
- J1 pad 2: (no net) -> GND
- J1 pad 20: (no net) -> Net-(J1-Pad20)
- J1 pad 21: (no net) -> AEN
- J1 pad 22: (no net) -> GND
- J1 pad 23: (no net) -> ~IOW
- J1 pad 24: (no net) -> GND
- J1 pad 25: (no net) -> ~IOR
- J1 pad 26: (no net) -> GND
- J1 pad 27: (no net) -> ~DACK
- J1 pad 28: (no net) -> GND
- J1 pad 29: (no net) -> DRQ
- J1 pad 3: (no net) -> D7
- J1 pad 30: (no net) -> GND
- J1 pad 31: (no net) -> IRQ
- J1 pad 32: (no net) -> GND
- J1 pad 33: (no net) -> A1
- J1 pad 34: (no net) -> Net-(J1-Pad34)
- J1 pad 35: (no net) -> A0
- J1 pad 36: (no net) -> GND
- J1 pad 37: (no net) -> ~CS
- J1 pad 38: (no net) -> GND
- J1 pad 39: (no net) -> ~DRIVE_ACTIVE
- J1 pad 4: (no net) -> GND
- J1 pad 40: (no net) -> GND
- J1 pad 5: (no net) -> D6
- J1 pad 6: (no net) -> GND
- J1 pad 7: (no net) -> D5
- J1 pad 8: (no net) -> GND
- J1 pad 9: (no net) -> D4
- U4 pad 34: CFG_LATCH -> CFG_DATA
Routing:
- added copper zone on B.Cu, net GND
- added copper zone on F.Cu, net GND
Other:
- outline, holes or cut-outs redrawn
- copper layers 2 -> 4
