File: XTA-35/XTA-35.sch (KiCad schematic (older format))
At the start: 30 parts, among them J1 XTA_Connector, J2 IBM_8bit_DBA, J3 XTA Power, J4 LED, J5 Debug, SW1 Config, SW2 Boot Internal, SW3 Reset, U1 74LVC245, U2 74LVC245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

Commit message: A bit more board/footprint work.
Parts:
- J1: footprint (none) -> Connector_PinHeader_2.54mm:PinHeader_2x20_P2.54mm_Horizontal
- J3: footprint (none) -> w_conn_pc:conn_hdd_15-24-4441
Changed lines of the file:
@@
 F 0 "J1" H 1650 3165 50  0000 C CNN
 F 1 "XTA_Connector" H 1650 3074 50  0000 C CNN
-F 2 "" H 1650 3050 50  0001 C CNN
+F 2 "Connector_PinHeader_2.54mm:PinHeader_2x20_P2.54mm_Horizontal" H 1650 3050 50  0001 C CNN
 F 3 "" H 1650 3050 50  0001 C CNN
 	1    1650 2000
@@
 F 0 "J3" H 768 7367 50  0000 C CNN
 F 1 "XTA Power" H 768 7276 50  0000 C CNN
-F 2 "" H 850 7050 50  0001 C CNN
+F 2 "w_conn_pc:conn_hdd_15-24-4441" H 850 7050 50  0001 C CNN
 F 3 "~" H 850 7050 50  0001 C CNN
 	1    850  7050
