File: XTA-35-TH/XTA-35-TH.sch (KiCad schematic (older format))
At the start: 36 parts, among them J1 XTA_Connector, J2 XTA Power, J3 LED, J4 SD0, J5 SD1, J6 Debug, SW1 Config, SW2 Boot Internal, SW3 Reset, U1 74LVC245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

Commit message: Added a couple of TODO's to XTA drive schematic.
Other:
- note added: "TODO: A-B needs to be \ntied high, or signal \ndirections reversed."
- note added: "TODO: Signal directions \nneed to be reversed. Also\nadd pulldown to DATA_DIR\nto be sure of direction on\npower-up."
- note added: "The PICO already has a 47uF cap on both the 5v and 3.3v\nside of the regulator, so no bulk capacitor is\nincluded in this design."
- note removed: "The PICO already has a 47uF cap on both the 5v and 3.3v\nside of the regulator, so none is included in this design."
Changed lines of the file:
@@
 Wire Wire Line
 	8500 4650 8700 4650
-Text Notes 7000 6850 0    39   ~ 0
+Text Notes 7000 6950 0    39   ~ 0
 On GP26-28, there is a clamp diode\nto 3.3v, should one be needed.
 Wire Wire Line
@@
 Text GLabel 8050 3850 0    50   Input ~ 0
 SD0_CS
-Text Notes 7000 6700 0    39   ~ 0
-The PICO already has a 47uF cap on both the 5v and 3.3v\nside of the regulator, so none is included in this design.
+Text Notes 7000 6750 0    39   ~ 0
+The PICO already has a 47uF cap on both the 5v and 3.3v\nside of the regulator, so no bulk capacitor is\nincluded in this design.
 Text GLabel 8050 3550 0    50   Input ~ 0
 CFG_DATA
@@
 Text Label 9100 6100 1    30   ~ 0
 SWCLK
+Text Notes 2300 5800 0    118  ~ 0
+TODO: A-B needs to be \ntied high, or signal \ndirections reversed.
+Text Notes 600  4850 0    118  ~ 0
+TODO: Signal directions \nneed to be reversed. Also\nadd pulldown to DATA_DIR\nto be sure of direction on\npower-up.
 $EndSCHEMATC

Commit message: Reorder Pico pins and fix direction of 245's.
Parts:
- removed R3: 10K, Resistor_SMD:R_1206_3216Metric, symbol Device:R
- added R4: 10K, Resistor_SMD:R_1206_3216Metric, symbol Device:R
- J6: value Debug -> DEBUG; footprint Connector_PinHeader_2.54mm:PinHeader_1x06_P2.54mm_Vertical -> Connector_PinHeader_2.54mm:PinHeader_1x03_P2.54mm_Vertical; symbol Connector_Generic:Conn_01x06 -> Connector_Generic:Conn_01x03
- renumbered R4 to R3
Connections:
- net A0: now also U2.17 (B1); no longer U2.2 (A0)
- net A0_3V3: now also U2.3 (A1), U5.21 (GP16); no longer U2.18 (B0), U5.16 (GP12)
- net A1: now also U2.18 (B0); no longer U2.3 (A1)
- net A1_3V3: now also U2.2 (A0), U5.22 (GP17); no longer U2.17 (B1), U5.17 (GP13)
- net AEN: now also U2.14 (B4); no longer U2.4 (A2)
- net AEN_3V3: now also U2.6 (A4), U5.25 (GP19); no longer U2.16 (B2), U5.19 (GP14)
- net CFG_CLK: now also U5.7 (GP5); no longer J6.4 (Pin_4), U5.2 (GP1)
- net CFG_DATA: now also U5.9 (GP6)
- net CFG_LATCH: now also J5.2 (CS), U5.6 (GP4); no longer J4.2 (CS), U5.4 (GP2)
- net D0: now also U1.18 (B0); no longer U1.2 (A0)
- net D0_3V3: now also U1.2 (A0), U5.11 (GP8); no longer U1.18 (B0), U5.6 (GP4)
- net D1: now also U1.17 (B1); no longer U1.3 (A1)
- net D1_3V3: now also U1.3 (A1), U5.12 (GP9); no longer U1.17 (B1), U5.7 (GP5)
- net D2: now also U1.16 (B2); no longer U1.4 (A2)
- net D2_3V3: now also U1.4 (A2), U5.14 (GP10); no longer U1.16 (B2), U5.9 (GP6)
- net D3: now also U1.15 (B3); no longer U1.5 (A3)
- net D3_3V3: now also U1.5 (A3), U5.15 (GP11); no longer U1.15 (B3), U5.10 (GP7)
- net D4: now also U1.14 (B4); no longer U1.6 (A4)
- net D4_3V3: now also U1.6 (A4), U5.16 (GP12); no longer U1.14 (B4), U5.11 (GP8)
- net D5: now also U1.13 (B5); no longer U1.7 (A5)
- net D5_3V3: now also U1.7 (A5), U5.17 (GP13); no longer U1.13 (B5), U5.12 (GP9)
- net D6: now also U1.12 (B6); no longer U1.8 (A6)
- net D6_3V3: now also U1.8 (A6), U5.19 (GP14); no longer U1.12 (B6), U5.14 (GP10)
- net D7: now also U1.11 (B7); no longer U1.9 (A7)
- net D7_3V3: now also U1.9 (A7), U5.20 (GP15); no longer U1.11 (B7), U5.15 (GP11)
- net DATA_DIR: now also U5.10 (GP7), R4.1; no longer U5.29 (GP22)
- net GND: now also R4.2; no longer J6.5 (Pin_5)
- net SPI_RX: now also U5.1 (GP0); no longer U5.21 (GP16)
- net SPI_SCK: now also U5.4 (GP2); no longer U5.24 (GP18)
- net SPI_TX: now also U5.5 (GP3); no longer U5.25 (GP19)
- net SWCLK: now also J6.1 (Pin_1); no longer J6.3 (Pin_3)
- net SWDIO: now also J6.3 (Pin_3); no longer J6.1 (Pin_1)
- net ~CS: now also U2.13 (B5); no longer U2.6 (A4)
- net ~CS~_3V3: now also U2.7 (A5), U5.24 (GP18); no longer U2.14 (B4), U5.31 (GP26)
- net ~DACK: now also U2.15 (B3); no longer U2.5 (A3)
- net ~DACK~_3V3: now also U2.5 (A3), U5.29 (GP22); no longer U2.15 (B3), U5.20 (GP15)
- net ~IOR: now also U2.12 (B6); no longer U2.8 (A6)
- net ~IOR~_3V3: now also U2.8 (A6); no longer U2.12 (B6)
- net ~IOW: now also U2.11 (B7); no longer U2.9 (A7)
- net ~IOW~_3V3: now also U2.9 (A7), U5.27 (GP21); no longer U2.11 (B7), U5.22 (GP17)
- net ~RESET: now also U2.16 (B2); no longer U2.7 (A5)
- net ~RESET~_3V3: now also U2.4 (A2), U5.31 (GP26); no longer U2.13 (B5), U5.27 (GP21)
- removed net DBG_RX: J6.6 (Pin_6), U5.1 (GP0)
- removed net SD1_CS: J5.2 (CS), U5.5 (GP3)
- new net SD0_CS: J4.2 (CS), U5.2 (GP1)
Other:
- note removed: "TODO: A-B needs to be \ntied high, or signal \ndirections reversed."
- note removed: "TODO: Signal directions \nneed to be reversed. Also\nadd pulldown to DATA_DIR\nto be sure of direction on\npower-up."
- moved on the sheet: SW3, U1
